Commit message: Fixed the bridge params Gave launch option and default to world uncommented ros2_control stuff Single rviz launch and rviz file Cleaned lidar xacro

File: urdf/lidar.xacro (robot description, xacro)
@@ -2,20 +2,17 @@
 <robot xmlns:xacro="http://www.ros.org/wiki/xacro" >
     <xacro:include filename="params.xacro" />
-    <material name="black">
+    <material name="lidar_black">
         <color rgba="0 0 0 1"/>
     </material>
-    <material name="blue">
+    <material name="lidar_blue">
         <color rgba="0.2 0.2 1 1"/>
     </material>
-    <xacro:property name="my_x_origin" value="${chassis_length/2}" />
-    <xacro:property name="my_y_origin" value="${-chassis_width/2}" />
-    <xacro:property name="my_z_origin" value="${chassis_height - drive_wheel_radius + chassis_Z_offset}" />
-    <xacro:property name="my_x_length" value="0.05" />
-    <xacro:property name="my_y_length" value="0.05" />
-    <xacro:property name="my_z_length" value="0.293" />
+    <xacro:property name="lidar_pole_x_origin" value="${chassis_length/2}" />
+    <xacro:property name="lidar_pole_y_origin" value="${-chassis_width/2}" />
+    <xacro:property name="lidar_pole_z_origin" value="${chassis_height - drive_wheel_radius + chassis_Z_offset}" />
     <joint name="lidar_mount_joint" type="fixed">
         <parent link="base_link"/>
         <child link="lidar_mount_link"/>
-        <origin xyz = "${my_x_origin-my_x_length/2 + chassis_X_offset} ${my_y_origin+my_y_length/2} ${my_z_origin + my_z_length/2}"/>
+        <origin xyz = "${lidar_pole_x_origin-lidar_pole_length/2 + chassis_X_offset} ${lidar_pole_y_origin+lidar_pole_width/2} ${lidar_pole_z_origin + lidar_pole_height/2}"/>
     </joint>
     <link name="lidar_mount_link">
@@ -23,16 +20,16 @@
             <origin xyz = "0 0 0"/>
             <geometry>
-                <box size="${my_x_length} ${my_y_length} ${my_z_length}"/>
+                <box size="${lidar_pole_length} ${lidar_pole_width} ${lidar_pole_height}"/>
             </geometry>
-            <material name="black"/>
+            <material name="lidar_black"/>
         </visual>
         <collision>
             <origin xyz = "0 0 0"/>
             <geometry>
-                <box size="${my_x_length} ${my_y_length} ${my_z_length}"/>
+                <box size="${lidar_pole_length} ${lidar_pole_width} ${lidar_pole_height}"/>
             </geometry>
-            <material name="black"/>
+            <material name="lidar_black"/>
         </collision>
-        <xacro:inertial_box mass="0.1" x="${my_x_length}" y="${my_y_length}" z="${my_z_length}">
+        <xacro:inertial_box mass="0.1" x="${lidar_pole_length}" y="${lidar_pole_width}" z="${lidar_pole_height}">
             <origin xyz="0 0 0" rpy="0 0 0"/>
         </xacro:inertial_box>
@@ -41,50 +38,22 @@
         <parent link="lidar_mount_link"/>
         <child link="laser"/>
-        <origin xyz = "0 0 0.167"/> <!--half the height of the mount + half the height of the lidar itself (0.293+0.04)/2-->
+        <origin xyz = "0 0 ${(lidar_pole_height+lidar_sensor_height)/2}"/> <!--half the height of the mount + half the height of the lidar itself -->
     </joint>
     <link name="laser">
         <visual>
             <geometry>
-                <cylinder radius="0.05" length="0.04"/>
+                <cylinder radius="${lidar_sensor_radius}" length="${lidar_sensor_radius}"/>
             </geometry>
-            <material name="blue"/>
+            <material name="lidar_blue"/>
         </visual>
         <collision>
             <geometry>
-                <cylinder radius="0.05" length="0.04"/>
+                <cylinder radius="${lidar_sensor_radius}" length="${lidar_sensor_radius}"/>
             </geometry>
         </collision>
-        <xacro:inertial_cylinder mass="0.1" length="0.04" radius="0.05">
-            <origin xyz="0 0 0.167" rpy="0 0 0"/>
+        <xacro:inertial_cylinder mass="0.1" radius="${lidar_sensor_radius}" length="${lidar_sensor_radius}" >
+            <origin xyz="0 0 ${(lidar_pole_height+lidar_sensor_height)/2}" rpy="0 0 0"/>
         </xacro:inertial_cylinder>
     </link>
-    <!-- <joint name="laser_joint" type="fixed">
-        <parent link="chassis"/>
-        <child link="laser_frame"/>
-        <origin xyz="0.122 0 0.212" rpy="0 0 0"/>
-    </joint>
-    <link name="laser_frame">
-        <visual>
-            <geometry>
-                <box radius="0.05" length="0.04"/>
-            </geometry>
-            <material name="black"/>
-        </visual>
-        <visual>
-            <origin xyz="${chassis_length/2 - 0.1} ${-chassis_width/2} -0.05"/>
-            <geometry>
-                <cylinder radius="0.01" length="0.1"/>
-            </geometry>
-            <material name="black"/>
-        </visual>
-        <collision>
-            <geometry>
-                <cylinder radius="0.05" length="0.04"/>
-            </geometry>
-        </collision>
-        <xacro:inertial_cylinder mass="0.1" length="0.04" radius="0.05">
-            <origin xyz="0 0 0" rpy="0 0 0"/>
-        </xacro:inertial_cylinder>
-    </link> -->
     <gazebo reference="laser">
         <material>Gazebo/blue</material>

File: urdf/params.xacro (robot description, xacro)
@@ -17,3 +17,9 @@
     <xacro:property name="caster_wheels_F_X_offset" value="0.35" />
     <xacro:property name="caster_wheels_R_X_offset" value="-0.4" />
+    <!--LIDAR-->
+    <xacro:property name="lidar_pole_height" value="0.293" />
+    <xacro:property name="lidar_pole_width" value="0.0635" />
+    <xacro:property name="lidar_pole_length" value="0.0635" />
+    <xacro:property name="lidar_sensor_height" value="0.02794" />
+    <xacro:property name="lidar_sensor_radius" value="0.0635" />
 </robot>
